Commit message: wheel radius, controller/planner changes (implemented for some time, not pushed until now)

File: husky_description/urdf/husky.urdf.xacro (robot description, xacro)
@@ -40,5 +40,5 @@
   <!-- Wheel Properties -->
   <xacro:property name="wheel_length" value="0.1143" />
-  <xacro:property name="wheel_radius" value="0.17775" />
+  <xacro:property name="wheel_radius" value="0.164" />
   <xacro:macro name="husky_robot">
     <!-- Base link is the center of the robot's bottom plate -->

Commit message: Increasing oscillation_timeout.

File: husky_description/urdf/husky.urdf.xacro (robot description, xacro)
@@ -66,5 +66,5 @@
     <link name="base_footprint"/>
     <joint name="base_footprint_joint" type="fixed">
-      <origin xyz="0 0 ${wheel_vertical_offset - wheel_radius}" rpy="0 0 0" />
+      <origin xyz="0 0 ${ (wheel_vertical_offset - wheel_radius) }" rpy="0 0 0" />
       <parent link="base_link" />
       <child link="base_footprint" />
