Commit message: updated top_plate to use an arg

File: husky_description/urdf/decorations.urdf.xacro (robot description, xacro)
@@ -79,5 +79,6 @@
       <child link="rear_bumper_link" />
     </joint>
-    <xacro:if value="$(optenv HUSKY_TOP_PLATE_ENABLED true)">
+    <xacro:if value="$(arg top_plate_enabled)">
+    <!--<xacro:if value="$(optenv HUSKY_TOP_PLATE_ENABLED true)"> -->
       <!-- Spawn the top plate -->
       <link name="top_plate_link">

Commit message: Remove top_plate_enabled substitution arg

File: husky_description/urdf/decorations.urdf.xacro (robot description, xacro)
@@ -79,34 +79,31 @@
       <child link="rear_bumper_link" />
     </joint>
-    <xacro:if value="$(arg top_plate_enabled)">
-    <!--<xacro:if value="$(optenv HUSKY_TOP_PLATE_ENABLED true)"> -->
-      <!-- Spawn the top plate -->
-      <link name="top_plate_link">
-        <visual>
-          <origin xyz="0 0 0" rpy="0 0 0" />
-          <geometry>
-            <mesh filename="package://husky_description/meshes/top_plate.dae" />
-          </geometry>
-        </visual>
-        <collision>
-          <origin xyz="0 0 0" rpy="0 0 0"/>
-          <geometry>
-            <mesh filename="package://husky_description/meshes/top_plate.dae" />
-          </geometry>
-        </collision>
-        <collision>
-          <!-- Extra collision tag for widgets on top plate -->
-          <geometry>
-            <box size="0.32 0.41 0.09" rpy="0 0 0"/>
-          </geometry>
-        </collision>
-      </link>
-      <!-- Attach top plate -->
-      <joint name="top_plate_joint" type="fixed">
-        <parent link="base_link" />
-        <child link="top_plate_link"/>
-        <origin xyz="0.0812 0 0.245" rpy="0 0 0"/>
-      </joint>
-    </xacro:if>
+    <!-- Spawn the top plate -->
+    <link name="top_plate_link">
+      <visual>
+        <origin xyz="0 0 0" rpy="0 0 0" />
+        <geometry>
+          <mesh filename="package://husky_description/meshes/top_plate.dae" />
+        </geometry>
+      </visual>
+      <collision>
+        <origin xyz="0 0 0" rpy="0 0 0"/>
+        <geometry>
+          <mesh filename="package://husky_description/meshes/top_plate.dae" />
+        </geometry>
+      </collision>
+      <collision>
+        <!-- Extra collision tag for widgets on top plate -->
+        <geometry>
+          <box size="0.32 0.41 0.09" rpy="0 0 0"/>
+        </geometry>
+      </collision>
+    </link>
+    <!-- Attach top plate -->
+    <joint name="top_plate_joint" type="fixed">
+      <parent link="base_link" />
+      <child link="top_plate_link"/>
+      <origin xyz="0.0812 0 0.245" rpy="0 0 0"/>
+    </joint>
   </xacro:macro>
 </robot>

Commit message: update husky description

File: husky_description/urdf/decorations.urdf.xacro (robot description, xacro)
@@ -79,31 +79,4 @@
       <child link="rear_bumper_link" />
     </joint>
-    <!-- Spawn the top plate -->
-    <link name="top_plate_link">
-      <visual>
-        <origin xyz="0 0 0" rpy="0 0 0" />
-        <geometry>
-          <mesh filename="package://husky_description/meshes/top_plate.dae" />
-        </geometry>
-      </visual>
-      <collision>
-        <origin xyz="0 0 0" rpy="0 0 0"/>
-        <geometry>
-          <mesh filename="package://husky_description/meshes/top_plate.dae" />
-        </geometry>
-      </collision>
-      <collision>
-        <!-- Extra collision tag for widgets on top plate -->
-        <geometry>
-          <box size="0.32 0.41 0.09" rpy="0 0 0"/>
-        </geometry>
-      </collision>
-    </link>
-    <!-- Attach top plate -->
-    <joint name="top_plate_joint" type="fixed">
-      <parent link="base_link" />
-      <child link="top_plate_link"/>
-      <origin xyz="0.0812 0 0.245" rpy="0 0 0"/>
-    </joint>
   </xacro:macro>
 </robot>
